Commit message: rtabmap for livox

File: livox_laser_simulation_ros2/urdf/mid360.xacro (robot description, xacro)
@@ -4,5 +4,5 @@
   <xacro:property name="laser_min_range" value="0.1"/>
   <xacro:property name="laser_max_range" value="200.0"/>
-  <xacro:property name="samples" value="40000"/>
+  <xacro:property name="samples" value="5000"/>
   <xacro:property name="resolution" value="0.002"/>
   <xacro:property name="noise_mean" value="0.0"/>
@@ -37,5 +37,5 @@
         <pose>0 0 0 0 0 0</pose>
         <visualize>true</visualize>
-        <update_rate>10</update_rate>
+        <update_rate>20</update_rate>
         <!-- This ray plgin is only for visualization. -->
         <plugin name="${name}_plugin" filename="libros2_livox.so">

File: robots/descriptions/go2_description/xacro/camera_gazebo.xacro (robot description, xacro)
@@ -10,6 +10,6 @@
           <horizontal_fov>1.57</horizontal_fov>
           <image>
-            <width>1280</width>
-            <height>720</height>
+            <width>640</width>
+            <height>480</height>
           </image>
           <clip>
@@ -24,5 +24,5 @@
         </camera>
         <always_on>1</always_on>
-        <update_rate>30</update_rate>
+        <update_rate>40</update_rate>
         <visualize>0</visualize>
       </sensor>
@@ -32,6 +32,6 @@
           <horizontal_fov>1.57</horizontal_fov>
           <image>
-            <width>1280</width>
-            <height>720</height>
+            <width>640</width>
+            <height>480</height>
             <format>RGB_INT8</format>
           </image>
@@ -47,5 +47,5 @@
         </camera>
         <always_on>1</always_on>
-        <update_rate>30</update_rate>
+        <update_rate>40</update_rate>
         <visualize>1</visualize>
       </sensor>
@@ -55,6 +55,6 @@
           <horizontal_fov>1.57</horizontal_fov>
           <image>
-            <width>1280</width>
-            <height>720</height>
+            <width>640</width>
+            <height>480</height>
             <format>L_INT8</format>
           </image>
@@ -70,5 +70,5 @@
         </camera>
         <always_on>1</always_on>
-        <update_rate>1</update_rate>
+        <update_rate>40</update_rate>
         <visualize>0</visualize>
       </sensor>
@@ -78,6 +78,6 @@
           <horizontal_fov>1.57</horizontal_fov>
           <image>
-            <width>1280</width>
-            <height>720</height>
+            <width>640</width>
+            <height>480</height>
             <format>L_INT8</format>
           </image>
@@ -93,5 +93,5 @@
         </camera>
         <always_on>1</always_on>
-        <update_rate>1</update_rate>
+        <update_rate>40</update_rate>
         <visualize>0</visualize>
       </sensor>
@@ -101,7 +101,7 @@
       <plugin name="${camera_name}" filename="librealsense_gazebo_plugin.so">
         <prefix>${camera_name}</prefix>
-        <depthUpdateRate>15.0</depthUpdateRate>
-        <colorUpdateRate>15.0</colorUpdateRate>
-        <infraredUpdateRate>1.0</infraredUpdateRate>
+        <depthUpdateRate>30.0</depthUpdateRate>
+        <colorUpdateRate>30.0</colorUpdateRate>
+        <infraredUpdateRate>30.0</infraredUpdateRate>
         <depthTopicName>aligned_depth_to_color/image_raw</depthTopicName>
         <depthCameraInfoTopicName>depth/camera_info</depthCameraInfoTopicName>
